File: Documentation/circuit_diagram_for_final.kicad_sch (KiCad schematic)
At the start: 6 parts, among them SW1 SW_SPST, SW2 RotaryEncoder_Switch, U1 MOUDLE-SEEEDUINO-XIAO-ESP32C3

Commit message: forgot to add accelerometer
Parts:
- added OLED1: ~, symbol 512_final_OLED_Accelerometer_symbols:ADXL345 Accelerometer
Connections:
- net at BT1.2 (-), D1.2 (GND), OLED.2 (GND)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: now also OLED1.1 (GND)
- net at D1.3 (VDD), OLED.1 (VCC), SW1.1 (A)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: now also OLED1.2 (VCC)
- net at OLED.4 (SDA), U1.5 (PA8_A4_D4_SDA): now also OLED1.7 (SDA)
- net at OLED.3 (SCL), U1.6 (PA9_A5_D5_SCL): now also OLED1.8 (SCL)
Changed lines of the file:
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@@
+	)
+	(junction
+		(at 167.64 85.09)
+		(diameter 0)
+		(color 0 0 0 0)
+	)
+	(junction
+		(at 111.76 100.33)
+		(diameter 0)
+		(color 0 0 0 0)
+	)
+	(junction
+		(at 170.18 88.9)
+		(diameter 0)
+		(color 0 0 0 0)
+	)
+	(junction
+		(at 113.03 96.52)
+		(diameter 0)
+		(color 0 0 0 0)
 	)
 	(junction
@@
 	(wire
 		(pts
+			(xy 111.76 46.99) (xy 111.76 100.33)
+		)
+		(stroke
+			(width 0)
+			(type default)
+		)
+	)
+	(wire
+		(pts
+			(xy 170.18 88.9) (xy 175.26 88.9)
+		)
+		(stroke
+			(width 0)
+			(type default)
+		)
+	)
+	(wire
+		(pts
+			(xy 200.66 44.45) (xy 113.03 44.45)
+		)
+		(stroke
+			(width 0)
+			(type default)
+		)
+	)
+	(wire
+		(pts
 			(xy 219.71 76.2) (xy 165.1 76.2)
 		)
@@
 	(wire
 		(pts
+			(xy 167.64 29.21) (xy 167.64 85.09)
+		)
+		(stroke
+			(width 0)
+			(type default)
+		)
+	)
+	(wire
+		(pts
+			(xy 167.64 85.09) (xy 168.91 85.09)
+		)
+		(stroke
+			(width 0)
+			(type default)
+		)
+	)
+	(wire
+		(pts
+			(xy 200.66 29.21) (xy 167.64 29.21)
+		)
+		(stroke
+			(width 0)
+			(type default)
+		)
+	)
+	(wire
+		(pts
 			(xy 171.45 63.5) (xy 171.45 92.71)
 		)
@@
 	(wire
 		(pts
+			(xy 111.76 100.33) (xy 114.3 100.33)
+		)
+		(stroke
+			(width 0)
+			(type default)
+		)
+	)
+	(wire
+		(pts
 			(xy 167.64 100.33) (xy 163.83 100.33)
 		)
@@
 	(wire
 		(pts
+			(xy 170.18 31.75) (xy 170.18 88.9)
+		)
+		(stroke
+			(width 0)
+			(type default)
+		)
+	)
+	(wire
+		(pts
 			(xy 200.66 96.52) (xy 219.71 96.52)
 		)
@@
 	(wire
 		(pts
+			(xy 200.66 31.75) (xy 170.18 31.75)
+		)
+		(stroke
+			(width 0)
+			(type default)
+		)
+	)
+	(wire
+		(pts
 			(xy 203.2 124.46) (xy 203.2 102.87)
 		)
@@
 	(wire
 		(pts
-			(xy 166.37 85.09) (xy 168.91 85.09)
+			(xy 166.37 85.09) (xy 167.64 85.09)
 		)
 		(stroke
@@
 	(wire
 		(pts
-			(xy 110.49 100.33) (xy 114.3 100.33)
+			(xy 110.49 100.33) (xy 111.76 100.33)
 		)
 		(stroke
@@
 	(wire
 		(pts
-			(xy 163.83 88.9) (xy 175.26 88.9)
+			(xy 163.83 88.9) (xy 170.18 88.9)
+		)
+		(stroke
+			(width 0)
+			(type default)
+		)
+	)
+	(wire
+		(pts
+			(xy 113.03 96.52) (xy 114.3 96.52)
 		)
 		(stroke
@@
 	(wire
 		(pts
+			(xy 200.66 46.99) (xy 111.76 46.99)
+		)
+		(stroke
+			(width 0)
+			(type default)
+		)
+	)
+	(wire
+		(pts
 			(xy 163.83 85.09) (xy 165.1 85.09)
 		)
@@
 	(wire
 		(pts
-			(xy 106.68 96.52) (xy 114.3 96.52)
+			(xy 106.68 96.52) (xy 113.03 96.52)
 		)
 		(stroke
@@
 	(wire
 		(pts
+			(xy 113.03 44.45) (xy 113.03 96.52)
+		)
+		(stroke
+			(width 0)
+			(type default)
+		)
+	)
+	(wire
+		(pts
 			(xy 167.64 124.46) (xy 167.64 100.33)
 		)
@@
 		)
 	)
+	(symbol
+		(lib_id "512_final_OLED_Accelerometer_symbols:ADXL345 Accelerometer")
+		(at 203.2 27.94 0)
+		(unit 1)
+		(exclude_from_sim no)
+		(in_bom yes)
+		(on_board yes)
+		(dnp no)
+		(fields_autoplaced yes)
+		(property "Reference" "OLED1"
+			(at 1224.28 -424.8151 0)
+			(effects
+				(font
+					(size 1.27 1.27)
+				)
+				(justify left)
+			)
+		)
+		(property "Value" "~"
+			(at 1224.28 -422.2751 0)
+			(effects
+				(font
+					(size 1.27 1.27)
+				)
+				(justify left)
+			)
+		)
+		(property "Footprint" ""
+			(at 203.2 27.94 0)
+			(effects
+				(font
+					(size 1.27 1.27)
+				)
+				(hide yes)
+			)
+		)
+		(property "Datasheet" ""
+			(at 203.2 27.94 0)
+			(effects
+				(font
+					(size 1.27 1.27)
+				)
+				(hide yes)
+			)
+		)
+		(property "Description" ""
+			(at 203.2 27.94 0)
+			(effects
+				(font
+					(size 1.27 1.27)
+				)
+				(hide yes)
+			)
+		)
+		(pin "4"
+		)
+		(pin "5"
+		)
+		(pin "1"
+		)
+		(pin "1"
+		)
+		(pin "1"
+		)
+		(pin "1"
+		)
+		(pin "6"
+		)
+		(pin "1"
+		)
+		(pin "1"
+		)
+		(pin "2"
+		)
+		(pin "3"
+		)
+		(pin "7"
+		)
+		(pin "8"
+		)
+		(instances
+			(project ""
+				(path "/08afefe6-1bfd-4a44-a180-3505e1895b3a"
+					(reference "OLED1")
+					(unit 1)
+				)
+			)
+		)
+	)
